File: LED_MATRIX_V2.0.kicad_pcb (KiCad board)
At the start: 2 copper layers, 71.8 x 40.7 mm, 31 parts, among them U1 ATTINY85-20PU

Commit message: updated the new logo
Parts:
- removed the G*** at (173.4, 99.7)
- added G***: LOGO, logo_Footprints:imt_new3, B.Cu at (171.5, 97.6)
